File: PID_Board/PID_Board.kicad_pcb (KiCad board)
At the start: 2 copper layers, 250 x 100 mm, 226 parts, among them J1 Axis_Mon, J2 IMU_GY521, J4 UPDI, J5 ESC_4in1, J6 ELRS_RX, J7 UPDI2, Q1 2N7000, Q2 2N7000, Q3 2N7000, U1 ATtiny1614-SS, U10 Pololu D24V5F5, U101 MCP6004, U102 TL431ACLPG, U2 74HC138, U201 MCP6004, U202 MCP6004, U3 ATtiny1614-SS, U301 MCP6004, U302 MCP6004, U4 MCP4822, U401 MCP6004, U402 MCP6004, U5 MCP4822, U6 MCP4822, U7 MCP4822, U8 MCP4822, U9 CD4066BE

Commit message: PID_Board THT: add ARM/I_HOLD pulldowns, silk cleanup, JLC/PCBWay fab export
- R24/R25 10k pulldowns on ARM and I_HOLD
- Silkscreen cleanup, board title, JLCJLCJLCJLC marker on back
- Fab export in fab/JLC_PCBWay_THT (gerbers, drill, BOM, CPL for U1/U3)
- KNOWN_ISSUES.md: 2N7000 level shifters (Q1-Q3) are marginal at ~3.4 V gate
  bias (max Vgs(th) 3 V); fallback is ZVN3306A in the same footprint
Parts:
- added R24: 10k, Resistor_THT:R_Axial_DIN0207_L6.3mm_D2.5mm_P10.16mm_Horizontal, F.Cu at (150.0, 23.5)
- added R25: 10k, Resistor_THT:R_Axial_DIN0207_L6.3mm_D2.5mm_P10.16mm_Horizontal, F.Cu at (150.0, 27.0)
Routing:
- net ARM: track 56.6 -> 78.0 mm
- net I_HOLD: track 57.0 -> 68.2 mm, vias 1 -> 2
Other:
- board text added: "ANALOG PID FC v1.0"
- board text added: "JLCJLCJLCJLC"

Commit message: PID_Board rev B: frame-mount layout (90x210 mm, 4-layer)
- Reshaped from 250x100 to 90x210 mm to fit the 5" frame: 30.5 stack and
  20x20 ESC stack holes with 3.4 mm copper-free standoff rings; tall parts
  kept out of the prop disks; GY-521 on J2 with the MPU-6050 over the CG
- Floorplan in bands (shim, roll, GY-521 + REF, pitch, yaw + control I/O +
  power over the ESC) with labelled per-axis tuning panels
- 4 layers: In1 GND plane, In2 +5V plane; routed with FreeRouting 2.5 plus
  a grid router for the last connections; DRC 0 errors, schematic parity clean
- Resistors moved to 7.62 mm pitch (still horizontal); ELRS header J6 moved
  to the front edge next to the shim MCU
- MOUNTING.md + mounting_plan.png, updated KNOWN_ISSUES, renders, 4-layer
  Gerbers/drill, grouped BOM and CPL
Parts:
- R1, R10, R101, R102, R103, R104, R11, R12, R13, R14, R15, R16, R17, R18, R19, R2, R20, R201, R202, R203, R204, R205, R206, R207, R208, R209, R21, R210, R211, R212, R213, R214, R215, R216, R217, R218, R219, R22, R220, R221, R23, R24, R25, R3, R301, R302, R303, R304, R305, R306, R307, R308, R309, R310, R311, R312, R313, R314, R315, R316, R317, R318, R319, R320, R321, R4, R401, R402, R403, R404, R405, R406, R407, R408, R409, R410, R411, R412, R413, R414, R5, R6, R7, R8, R9: footprint Resistor_THT:R_Axial_DIN0207_L6.3mm_D2.5mm_P10.16mm_Horizontal -> Resistor_THT:R_Axial_DIN0207_L6.3mm_D2.5mm_P7.62mm_Horizontal
- moved R413 223.9 mm to (76.8, 162.6)
- moved R411 209.0 mm to (80.3, 173.0)
- moved R414 206.4 mm to (78.7, 145.1)
- moved RV401 200.2 mm to (93.9, 183.4), turned to 90 degrees
- moved U402 199.4 mm to (95.9, 152.4), turned to -90 degrees
- moved C403 190.3 mm to (116.2, 173.0)
- moved TP402 188.7 mm to (99.9, 176.0)
- moved R412 184.7 mm to (90.2, 141.3), turned to 180 degrees
- moved D404 184.5 mm to (120.3, 195.3)
- moved RV403 182.9 mm to (106.6, 183.4), turned to 90 degrees
- moved C401 178.0 mm to (102.6, 166.7), turned to -90 degrees
- moved RV402 176.3 mm to (100.3, 183.4), turned to 90 degrees
- moved R405 174.1 mm to (135.3, 159.4), turned to 180 degrees
- moved R406 171.7 mm to (120.0, 165.7), turned to -90 degrees
- moved TP404 171.1 mm to (107.5, 176.0)
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Routing:
- net GND: track 906.1 -> 8.18 mm, vias 1 -> 0
- net +5V: track 763.4 -> 6.43 mm, vias 3 -> 1
- net ROLL_ANGLE: track 225.7 -> 23.5 mm, vias 3 -> 0
- net ROLL_RATE: track 199.0 -> 22.2 mm, vias 2 -> 0
- net YAW_RATE: track 51.7 -> 190.0 mm, vias 0 -> 3
- net YAW_RATE_CMD: track 50.9 -> 186.0 mm, vias 0 -> 1
- net ROLL_ANGLE_CMD: track 156.7 -> 35.4 mm
- net U_ROLL: track 293.0 -> 183.4 mm, vias 2 -> 8
- net VGND_C: track 286.8 -> 194.7 mm
- net /SCL_3V3: track 16.2 -> 94.9 mm, vias 0 -> 1
- net /CS_DAC5: track 87.2 -> 9.49 mm, vias 1 -> 0
- net U_YAW: track 215.6 -> 140.9 mm, vias 2 -> 4
- net Net-(D201-A): track 169.2 -> 98.0 mm
- net PITCH_RATE: track 147.6 -> 78.6 mm, vias 1 -> 0
- net Net-(U301A-+): track 77.5 -> 14.8 mm, vias 1 -> 0
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- added copper zone on In2.Cu, net +5V
- added copper zone on In1.Cu, net GND
- removed copper zone on B.Cu, net GND
- removed copper zone on F.Cu, net GND
Other:
- board size 250 x 100 mm -> 90 x 210 mm
- copper layers 2 -> 4
- board text added: "CRSF"
- board text added: "D"
- board text added: "EA"
- board text added: "ERR"
- board text added: "FRONT"
- board text added: "GYRO EXT"
- board text added: "Go"
- board text added: "I"
- board text added: "J1 SCOPE"
- board text added: "J4 UPDI"
- board text added: "J5 ESC"
- board text added: "J6 ELRS"
- board text added: "J7 UPDI2"
- board text added: "Kd"
- board text added: "Ki"
- board text added: "Kp"
- board text added: "LOOP EXT"
- board text added: "P"
- board text added: "PID_Board THT rev B"
- board text added: "PID_Board THT rev B 4-layer: In1 GND, In2 +5V"
- board text added: "PLT"
- board text added: "REF"
- board text added: "U"
- board text added: "U10 BUCK"
- board text added: "VGA"
- board text added: "VGB"
- board text added: "VGC"
- board text added: "VREF"
- board text added: "VSET"
- board text added: "XFB"
- board text added: "XSP"
- board text removed: "ANALOG PID FC v1.0"
- board text removed: "B+"
- board text removed: "B-"
- board text removed: "CG"
- board text removed: "CUR"
- board text removed: "DAC SHIM + REF"
- board text removed: "ESC cable"
- board text removed: "EXT"
- board text removed: "FRONT (remap in firmware)"
- board text removed: "GYRO"
- board text removed: "J1 AXIS MON"
- board text removed: "J2 GY-521"
- board text removed: "J4 UPDI MCU"
- board text removed: "J5 ESC 4in1"
- board text removed: "J6 ELRS RX"
- board text removed: "J7 UPDI ESC"
- board text removed: "JP201 LOOP SP"
- board text removed: "JP202 LOOP FB"
- board text removed: "JP301 LOOP SP"
- board text removed: "JP302 LOOP FB"
- board text removed: "JP401 LOOP SP"
- board text removed: "JP402 LOOP FB"
- board text removed: "M1"
- board text removed: "M2"
- board text removed: "M3"
- board text removed: "M4"
- board text removed: "PITCH PID"
- board text removed: "ROLL PID"
- board text removed: "RX"
- board text removed: "SEL"
- board text removed: "SHDN"
- board text removed: "SPARE"
- board text removed: "TX"
- board text removed: "U10 BUCK 5V"
- board text removed: "VIN"
- board text removed: "VOUT"
- board text removed: "YAW PID"

Commit message: U10: use cheap fixed-5V mini buck module wired to the existing header
- Value/BOM: 5V buck module (Teyleten 3A Mini DCDC Buck, 5.5-30V in, Amazon B0DKTMGBHL)
- MOUNTING.md: wiring IN+ -> pin 2, IN- -> pin 3, OUT+ -> pin 4; no copper change
- KNOWN_ISSUES: power section is 2S-4S; for 6S C25 needs a 35 V+ rating
- CHANGELOG rev B.1
Parts:
- U10: value Pololu D24V5F5 -> 5V buck module (Mini 5V 3A)
Changed lines of the file:
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@@
 			)
 		)
-		(property "Value" "Pololu D24V5F5"
+		(property "Value" "5V buck module (Mini 5V 3A)"
 			(at 0 10 0)
 			(layer "F.Fab")
