File: PID_Board/control_io.kicad_sch (KiCad schematic)
At the start: 18 parts, among them J5 ESC_4in1, J7 UPDI2, U10 Pololu D24V5F5, U3 ATtiny1614-SS, U9 CD4066BE

Commit message: PID_Board rev B: frame-mount layout (90x210 mm, 4-layer)
- Reshaped from 250x100 to 90x210 mm to fit the 5" frame: 30.5 stack and
  20x20 ESC stack holes with 3.4 mm copper-free standoff rings; tall parts
  kept out of the prop disks; GY-521 on J2 with the MPU-6050 over the CG
- Floorplan in bands (shim, roll, GY-521 + REF, pitch, yaw + control I/O +
  power over the ESC) with labelled per-axis tuning panels
- 4 layers: In1 GND plane, In2 +5V plane; routed with FreeRouting 2.5 plus
  a grid router for the last connections; DRC 0 errors, schematic parity clean
- Resistors moved to 7.62 mm pitch (still horizontal); ELRS header J6 moved
  to the front edge next to the shim MCU
- MOUNTING.md + mounting_plan.png, updated KNOWN_ISSUES, renders, 4-layer
  Gerbers/drill, grouped BOM and CPL
Parts:
- R15, R16, R17, R18, R19, R20, R21, R22: footprint Resistor_THT:R_Axial_DIN0207_L6.3mm_D2.5mm_P10.16mm_Horizontal -> Resistor_THT:R_Axial_DIN0207_L6.3mm_D2.5mm_P7.62mm_Horizontal
Changed lines of the file:
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@@
 			)
 		)
-		(property "Footprint" "Resistor_THT:R_Axial_DIN0207_L6.3mm_D2.5mm_P10.16mm_Horizontal"
+		(property "Footprint" "Resistor_THT:R_Axial_DIN0207_L6.3mm_D2.5mm_P7.62mm_Horizontal"
 			(at 172.72 124.46 90)
 			(hide yes)
@@
 			)
 		)
-		(property "Footprint" "Resistor_THT:R_Axial_DIN0207_L6.3mm_D2.5mm_P10.16mm_Horizontal"
+		(property "Footprint" "Resistor_THT:R_Axial_DIN0207_L6.3mm_D2.5mm_P7.62mm_Horizontal"
 			(at 182.88 130.81 0)
 			(hide yes)
@@
 			)
 		)
-		(property "Footprint" "Resistor_THT:R_Axial_DIN0207_L6.3mm_D2.5mm_P10.16mm_Horizontal"
+		(property "Footprint" "Resistor_THT:R_Axial_DIN0207_L6.3mm_D2.5mm_P7.62mm_Horizontal"
 			(at 172.72 139.7 90)
 			(hide yes)
@@
 			)
 		)
-		(property "Footprint" "Resistor_THT:R_Axial_DIN0207_L6.3mm_D2.5mm_P10.16mm_Horizontal"
+		(property "Footprint" "Resistor_THT:R_Axial_DIN0207_L6.3mm_D2.5mm_P7.62mm_Horizontal"
 			(at 182.88 146.05 0)
 			(hide yes)
@@
 			)
 		)
-		(property "Footprint" "Resistor_THT:R_Axial_DIN0207_L6.3mm_D2.5mm_P10.16mm_Horizontal"
+		(property "Footprint" "Resistor_THT:R_Axial_DIN0207_L6.3mm_D2.5mm_P7.62mm_Horizontal"
 			(at 172.72 154.94 90)
 			(hide yes)
@@
 			)
 		)
-		(property "Footprint" "Resistor_THT:R_Axial_DIN0207_L6.3mm_D2.5mm_P10.16mm_Horizontal"
+		(property "Footprint" "Resistor_THT:R_Axial_DIN0207_L6.3mm_D2.5mm_P7.62mm_Horizontal"
 			(at 182.88 161.29 0)
 			(hide yes)
@@
 			)
 		)
-		(property "Footprint" "Resistor_THT:R_Axial_DIN0207_L6.3mm_D2.5mm_P10.16mm_Horizontal"
+		(property "Footprint" "Resistor_THT:R_Axial_DIN0207_L6.3mm_D2.5mm_P7.62mm_Horizontal"
 			(at 172.72 170.18 90)
 			(hide yes)
@@
 			)
 		)
-		(property "Footprint" "Resistor_THT:R_Axial_DIN0207_L6.3mm_D2.5mm_P10.16mm_Horizontal"
+		(property "Footprint" "Resistor_THT:R_Axial_DIN0207_L6.3mm_D2.5mm_P7.62mm_Horizontal"
 			(at 182.88 176.53 0)
 			(hide yes)

Commit message: U10: use cheap fixed-5V mini buck module wired to the existing header
- Value/BOM: 5V buck module (Teyleten 3A Mini DCDC Buck, 5.5-30V in, Amazon B0DKTMGBHL)
- MOUNTING.md: wiring IN+ -> pin 2, IN- -> pin 3, OUT+ -> pin 4; no copper change
- KNOWN_ISSUES: power section is 2S-4S; for 6S C25 needs a 35 V+ rating
- CHANGELOG rev B.1
Parts:
- U10: value Pololu D24V5F5 -> 5V buck module (Mini 5V 3A)
Other:
- note added: "Power: VBAT (2S-4S via ESC harness) -> 1N5817 -> 5V buck module on U10 (IN+ pin 2, GND pin 3, OUT+ pin 4) -> +5V"
- note removed: "Power: VBAT (2S-4S via ESC harness) -> 1N5817 -> Pololu D24V5F5 -> +5V"
Changed lines of the file:
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@@
 		)
 	)
-	(text "Power: VBAT (2S-4S via ESC harness) -> 1N5817 -> Pololu D24V5F5 -> +5V"
+	(text "Power: VBAT (2S-4S via ESC harness) -> 1N5817 -> 5V buck module on U10 (IN+ pin 2, GND pin 3, OUT+ pin 4) -> +5V"
 		(exclude_from_sim no)
 		(at 20.32 99.06 0)
@@
 			)
 		)
-		(property "Value" "Pololu D24V5F5"
+		(property "Value" "5V buck module (Mini 5V 3A)"
 			(at 81.28 125.73 0)
 			(effects
